Commit message: Added Gazebo plugin to hold object in place once grasped Reduced arm weights Increased velocity limits

File: Models/kuka_iiwa_14_prismatic_gripper/ros/iiwa_gripper.urdf (robot description, URDF)
Before this commit: robot iiwa14_gripper::iiwa14, 13 links, 12 joints
Links:
- link base_link_link: mass 1.0 -> 0.5
- link gripper_left_link: mass 1.0 -> 0.1
- link gripper_right_link: mass 1.0 -> 0.1
- link iiwa_link_2: mass 4 -> 0.4
- link iiwa_link_3: mass 3 -> 0.3
- link iiwa_link_4: mass 2.7 -> 0.27
- link iiwa_link_5: mass 1.7 -> 0.17
- link iiwa_link_6: mass 1.8 -> 0.18
- link iiwa_link_7: mass 0.3 -> 0.03
